File: Audio.sch (KiCad schematic (older format))
At the start: 53 parts, among them J5 PJ-3270, J6 PJ-3270, J7 PJ-3270, U6 SSM2603, Y1 12.288Mhz

Commit message: Implement battery management
Very rough and needs some clenup
Parts:
- J5, J6, J7: symbol otter:PJ-3270 -> OtterCastAudioV2-rescue:PJ-3270-otter
- U6: symbol otter:SSM2603 -> OtterCastAudioV2-rescue:SSM2603-otter
Changed lines of the file:
@@
 BT-PCM-DOUT
 $Comp
-L otter:SSM2603 U6
+L OtterCastAudioV2-rescue:SSM2603-otter U6
 U 1 1 5FF6F21F
 P 5750 4050
@@
 $EndComp
 $Comp
-L otter:GND #PWR0205
+L OtterCastAudioV2-rescue:GND-otter #PWR0205
 U 1 1 5FF88FDC
 P 5850 5800
@@
 $EndComp
 $Comp
-L otter:GND #PWR0206
+L OtterCastAudioV2-rescue:GND-otter #PWR0206
 U 1 1 5FF8C63C
 P 6050 5800
@@
 $EndComp
 $Comp
-L S3-OLinuXino_Rev_A:GND #PWR?
+L OtterCastAudioV2-rescue:GND-S3-OLinuXino_Rev_A #PWR?
 U 1 1 5FF96B43
 P 4850 5150
@@
 Connection ~ 4750 5250
 $Comp
-L S3-OLinuXino_Rev_A:GND #PWR?
+L OtterCastAudioV2-rescue:GND-S3-OLinuXino_Rev_A #PWR?
 U 1 1 5FF96B59
 P 4650 5150
@@
 	4750 5250 4400 5250
 $Comp
-L S3-OLinuXino_Rev_A:GND #PWR?
+L OtterCastAudioV2-rescue:GND-S3-OLinuXino_Rev_A #PWR?
 U 1 1 5FF96B61
 P 4100 5050
@@
 	4100 5050 4200 5050
 $Comp
-L S3-OLinuXino_Rev_A:GND #PWR?
+L OtterCastAudioV2-rescue:GND-S3-OLinuXino_Rev_A #PWR?
 U 1 1 5FF96B68
 P 4100 5250
@@
 $EndComp
 $Comp
-L S3-OLinuXino_Rev_A:+3.3V #PWR?
+L OtterCastAudioV2-rescue:+3.3V-S3-OLinuXino_Rev_A #PWR?
 U 1 1 5FFB96F5
 P 4100 4550
@@
 Connection ~ 6750 2100
 $Comp
-L otter:GND #PWR0213
+L OtterCastAudioV2-rescue:GND-otter #PWR0213
 U 1 1 601BC91C
 P 6800 2400
@@
 Connection ~ 6750 2400
 $Comp
-L otter:GND #PWR0214
+L OtterCastAudioV2-rescue:GND-otter #PWR0214
 U 1 1 601C6C24
 P 6600 2000
@@
 	4850 1700 5150 1700
 $Comp
-L S3-OLinuXino_Rev_A:+3.0VA #PWR?
+L OtterCastAudioV2-rescue:+3.0VA-S3-OLinuXino_Rev_A #PWR?
 U 1 1 6023A1C9
 P 6600 1700
@@
 Connection ~ 4850 1700
 $Comp
-L S3-OLinuXino_Rev_A:+3.0VA #PWR?
+L OtterCastAudioV2-rescue:+3.0VA-S3-OLinuXino_Rev_A #PWR?
 U 1 1 6027AD71
 P 4250 1700
@@
 $EndComp
 $Comp
-L S3-OLinuXino_Rev_A:+3.0VA #PWR?
+L OtterCastAudioV2-rescue:+3.0VA-S3-OLinuXino_Rev_A #PWR?
 U 1 1 602F2215
 P 4250 2100
@@
 	6750 5400 6750 5350
 $Comp
-L otter:GND #PWR0231
+L OtterCastAudioV2-rescue:GND-otter #PWR0231
 U 1 1 60A50D39
 P 6800 5400
@@
 Connection ~ 6400 5100
 $Comp
-L otter:PJ-3270 J7
+L OtterCastAudioV2-rescue:PJ-3270-otter J7
 U 1 1 60B772BD
 P 9050 2900
@@
 $EndComp
 $Comp
-L otter:PJ-3270 J6
+L OtterCastAudioV2-rescue:PJ-3270-otter J6
 U 1 1 60B798B5
 P 8450 3400
@@
 $EndComp
 $Comp
-L otter:PJ-3270 J5
+L OtterCastAudioV2-rescue:PJ-3270-otter J5
 U 1 1 60B92BDF
 P 3200 3100
@@
 	2950 2500 2950 2450
 $Comp
-L S3-OLinuXino_Rev_A:+3.0VA #PWR?
+L OtterCastAudioV2-rescue:+3.0VA-S3-OLinuXino_Rev_A #PWR?
 U 1 1 60C3B44B
 P 2950 2200
@@
 $EndComp
 $Comp
-L otter:GND #PWR0295
+L OtterCastAudioV2-rescue:GND-otter #PWR0295
 U 1 1 5FE5C65A
 P 5850 6600
