File: MIPI.sch (KiCad schematic (older format))
At the start: 40 parts, among them J8 49F-1201GYD2NL, U1 AllWinner-S3(FBGA-234), Y2 32.768kHz, Y3 24MHz

Commit message: Implement battery management
Very rough and needs some clenup
Parts:
- J8: symbol otter:49F-1201GYD2NL -> OtterCastAudioV2-rescue:49F-1201GYD2NL-otter
- U1: symbol otter:AllWinner-S3(FBGA-234) -> OtterCastAudioV2-rescue:AllWinner-S3(FBGA-234)-otter
Changed lines of the file:
@@
 	2700 1900 2300 1900
 $Comp
-L S3-OLinuXino_Rev_A:GND #PWR?
+L OtterCastAudioV2-rescue:GND-S3-OLinuXino_Rev_A #PWR?
 U 1 1 621FAA13
 P 2000 1900
@@
 $EndComp
 $Comp
-L S3-OLinuXino_Rev_A:GND #PWR?
+L OtterCastAudioV2-rescue:GND-S3-OLinuXino_Rev_A #PWR?
 U 1 1 621FAA25
 P 2350 3900
@@
 $EndComp
 $Comp
-L S3-OLinuXino_Rev_A:+3.0VA #PWR?
+L OtterCastAudioV2-rescue:+3.0VA-S3-OLinuXino_Rev_A #PWR?
 U 1 1 621FAA2B
 P 2350 3700
@@
 $EndComp
 $Comp
-L S3-OLinuXino_Rev_A:+3.3V #PWR?
+L OtterCastAudioV2-rescue:+3.3V-S3-OLinuXino_Rev_A #PWR?
 U 1 1 621FAA43
 P 1900 2300
@@
 $EndComp
 $Comp
-L S3-OLinuXino_Rev_A:GND #PWR?
+L OtterCastAudioV2-rescue:GND-S3-OLinuXino_Rev_A #PWR?
 U 1 1 621FAA8A
 P 1200 4350
@@
 $EndComp
 $Comp
-L S3-OLinuXino_Rev_A:GND #PWR?
+L OtterCastAudioV2-rescue:GND-S3-OLinuXino_Rev_A #PWR?
 U 1 1 621FAA9B
 P 1550 4500
@@
 $EndComp
 $Comp
-L S3-OLinuXino_Rev_A:+3.3V #PWR?
+L OtterCastAudioV2-rescue:+3.3V-S3-OLinuXino_Rev_A #PWR?
 U 1 1 621FAAB0
 P 1200 4100
@@
 $EndComp
 $Comp
-L S3-OLinuXino_Rev_A:GND #PWR?
+L OtterCastAudioV2-rescue:GND-S3-OLinuXino_Rev_A #PWR?
 U 1 1 621FAAC7
 P 2550 5650
@@
 $EndComp
 $Comp
-L S3-OLinuXino_Rev_A:VCC-DDR #PWR?
+L OtterCastAudioV2-rescue:VCC-DDR-S3-OLinuXino_Rev_A #PWR?
 U 1 1 621FAAD2
 P 1550 4750
@@
 	2500 5200 2700 5200
 $Comp
-L S3-OLinuXino_Rev_A:GND #PWR?
+L OtterCastAudioV2-rescue:GND-S3-OLinuXino_Rev_A #PWR?
 U 1 1 621FAAF3
 P 2150 5400
@@
 $EndComp
 $Comp
-L S3-OLinuXino_Rev_A:+3.0VA #PWR?
+L OtterCastAudioV2-rescue:+3.0VA-S3-OLinuXino_Rev_A #PWR?
 U 1 1 621FAB39
 P 5950 5000
@@
 	4100 4400 4550 4400
 $Comp
-L S3-OLinuXino_Rev_A:GND #PWR?
+L OtterCastAudioV2-rescue:GND-S3-OLinuXino_Rev_A #PWR?
 U 1 1 621FAB92
 P 4800 3800
@@
 $EndComp
 $Comp
-L S3-OLinuXino_Rev_A:GND #PWR?
+L OtterCastAudioV2-rescue:GND-S3-OLinuXino_Rev_A #PWR?
 U 1 1 621FAB9A
 P 5350 3700
@@
 $EndComp
 $Comp
-L S3-OLinuXino_Rev_A:+3.3V #PWR?
+L OtterCastAudioV2-rescue:+3.3V-S3-OLinuXino_Rev_A #PWR?
 U 1 1 621FABA1
 P 5350 3400
@@
 $EndComp
 $Comp
-L S3-OLinuXino_Rev_A:+1.1V #PWRV?
+L OtterCastAudioV2-rescue:+1.1V-S3-OLinuXino_Rev_A #PWRV?
 U 1 1 621FABBF
 P 4800 3500
@@
 $EndComp
 $Comp
-L S3-OLinuXino_Rev_A:+3.3V_RTC #PWR?
+L OtterCastAudioV2-rescue:+3.3V_RTC-S3-OLinuXino_Rev_A #PWR?
 U 1 1 621FAC6A
 P 5950 4350
@@
 $EndComp
 $Comp
-L S3-OLinuXino_Rev_A:+3.3V #PWR?
+L OtterCastAudioV2-rescue:+3.3V-S3-OLinuXino_Rev_A #PWR?
 U 1 1 621FACF7
 P 4100 2200
@@
 $EndComp
 $Comp
-L otter:AllWinner-S3(FBGA-234) U?
+L OtterCastAudioV2-rescue:AllWinner-S3(FBGA-234)-otter U?
 U 5 1 67B22B9C
 P 3400 3600
@@
 	1150 3800 1150 3750
 $Comp
-L S3-OLinuXino_Rev_A:GND #PWR?
+L OtterCastAudioV2-rescue:GND-S3-OLinuXino_Rev_A #PWR?
 U 1 1 682228FC
 P 1100 3800
@@
 	4400 5200 4100 5200
 $Comp
-L S3-OLinuXino_Rev_A:GND #PWR?
+L OtterCastAudioV2-rescue:GND-S3-OLinuXino_Rev_A #PWR?
 U 1 1 68801614
 P 4600 5250
@@
 Connection ~ 4700 5150
 $Comp
-L S3-OLinuXino_Rev_A:GND #PWR?
+L OtterCastAudioV2-rescue:GND-S3-OLinuXino_Rev_A #PWR?
 U 1 1 6887244B
 P 4800 5250
@@
 	4700 5150 5050 5150
 $Comp
-L S3-OLinuXino_Rev_A:GND #PWR?
+L OtterCastAudioV2-rescue:GND-S3-OLinuXino_Rev_A #PWR?
 U 1 1 688B7D1F
 P 5350 5350
@@
 	5350 5350 5250 5350
 $Comp
-L S3-OLinuXino_Rev_A:GND #PWR?
+L OtterCastAudioV2-rescue:GND-S3-OLinuXino_Rev_A #PWR?
 U 1 1 688D2E39
 P 5350 5150
@@
 	5350 5150 5250 5150
 $Comp
-L S3-OLinuXino_Rev_A:GND #PWR?
+L OtterCastAudioV2-rescue:GND-S3-OLinuXino_Rev_A #PWR?
 U 1 1 688E06D9
 P 5950 5300
@@
 $EndComp
 $Comp
-L S3-OLinuXino_Rev_A:GND #PWR?
+L OtterCastAudioV2-rescue:GND-S3-OLinuXino_Rev_A #PWR?
 U 1 1 68934D4E
 P 4700 4900
@@
 $EndComp
 $Comp
-L S3-OLinuXino_Rev_A:GND #PWR?
+L OtterCastAudioV2-rescue:GND-S3-OLinuXino_Rev_A #PWR?
 U 1 1 6898A97A
 P 5550 4800
@@
 	5550 4800 5450 4800
 $Comp
-L S3-OLinuXino_Rev_A:GND #PWR?
+L OtterCastAudioV2-rescue:GND-S3-OLinuXino_Rev_A #PWR?
 U 1 1 6898A981
 P 5550 4600
@@
 	5950 4450 5950 4400
 $Comp
-L S3-OLinuXino_Rev_A:GND #PWR?
+L OtterCastAudioV2-rescue:GND-S3-OLinuXino_Rev_A #PWR?
 U 1 1 68A05AC3
 P 5950 4650
@@
 EPHY_SPD_LED
 $Comp
-L S3-OLinuXino_Rev_A:+3.3V #PWR?
+L OtterCastAudioV2-rescue:+3.3V-S3-OLinuXino_Rev_A #PWR?
 U 1 1 68ABBB53
 P 7750 1650
@@
 $EndComp
 $Comp
-L S3-OLinuXino_Rev_A:+3.3V #PWR?
+L OtterCastAudioV2-rescue:+3.3V-S3-OLinuXino_Rev_A #PWR?
 U 1 1 68AC8602
 P 7450 1650
@@
 $EndComp
 $Comp
-L S3-OLinuXino_Rev_A:GND #PWR?
+L OtterCastAudioV2-rescue:GND-S3-OLinuXino_Rev_A #PWR?
 U 1 1 68B013CC
 P 8450 2500
@@
 $EndComp
 $Comp
-L S3-OLinuXino_Rev_A:GND #PWR?
+L OtterCastAudioV2-rescue:GND-S3-OLinuXino_Rev_A #PWR?
 U 1 1 68B0DC25
 P 8450 2100
@@
 	8950 2250 9000 2250
 $Comp
-L S3-OLinuXino_Rev_A:GND #PWR?
+L OtterCastAudioV2-rescue:GND-S3-OLinuXino_Rev_A #PWR?
 U 1 1 68C73D5E
 P 9700 2100
@@
 $EndComp
 $Comp
-L S3-OLinuXino_Rev_A:GND #PWR?
+L OtterCastAudioV2-rescue:GND-S3-OLinuXino_Rev_A #PWR?
 U 1 1 68C80600
 P 9700 2500
@@
 $EndComp
 $Comp
-L S3-OLinuXino_Rev_A:GND #PWR?
+L OtterCastAudioV2-rescue:GND-S3-OLinuXino_Rev_A #PWR?
 U 1 1 68C8FA66
 P 7550 3150
@@
 Connection ~ 1600 4750
 $Comp
-L S3-OLinuXino_Rev_A:GND #PWR?
+L OtterCastAudioV2-rescue:GND-S3-OLinuXino_Rev_A #PWR?
 U 1 1 68D50852
 P 1550 5100
@@
 	9350 2500 9350 2550
 $Comp
-L otter:49F-1201GYD2NL J8
+L OtterCastAudioV2-rescue:49F-1201GYD2NL-otter J8
 U 1 1 60475CA8
 P 7550 2300
@@
 	7350 1350 7350 1200
 $Comp
-L S3-OLinuXino_Rev_A:GND #PWR?
+L OtterCastAudioV2-rescue:GND-S3-OLinuXino_Rev_A #PWR?
 U 1 1 60388407
 P 5100 4200
