File: OtterCastAudioV2.sch (KiCad schematic (older format))
At the start: 21 parts, among them J1 UART, J2 SD, U1 AllWinner-S3(FBGA-234)

Commit message: Implement battery management
Very rough and needs some clenup
Parts:
- U1: symbol otter:AllWinner-S3(FBGA-234) -> OtterCastAudioV2-rescue:AllWinner-S3(FBGA-234)-otter
Changed lines of the file:
@@
 $EndDescr
 $Comp
-L S3-OLinuXino_Rev_A:+3.3V #PWR046
+L OtterCastAudioV2-rescue:+3.3V-S3-OLinuXino_Rev_A #PWR046
 U 1 1 5D97B54A
 P 10450 3250
@@
 	10750 3400 10850 3400
 $Comp
-L S3-OLinuXino_Rev_A:GND #PWR047
+L OtterCastAudioV2-rescue:GND-S3-OLinuXino_Rev_A #PWR047
 U 1 1 57966C0E
 P 8100 10700
@@
 $EndComp
 $Comp
-L otter:GND #PWR0101
+L OtterCastAudioV2-rescue:GND-otter #PWR0101
 U 1 1 6253E6C2
 P 14050 8800
@@
 $EndComp
 $Comp
-L S3-OLinuXino_Rev_A:GND #PWR0102
+L OtterCastAudioV2-rescue:GND-S3-OLinuXino_Rev_A #PWR0102
 U 1 1 6253EB67
 P 12350 8800
@@
 	11250 8000 11250 8100
 $Comp
-L otter:GND #PWR0103
+L OtterCastAudioV2-rescue:GND-otter #PWR0103
 U 1 1 62D601B0
 P 12350 8400
@@
 $EndComp
 $Comp
-L otter:GND #PWR0104
+L OtterCastAudioV2-rescue:GND-otter #PWR0104
 U 1 1 62F7C4A4
 P 11050 8450
@@
 	11050 8200 12350 8200
 $Comp
-L S3-OLinuXino_Rev_A:+3.3V #PWR0105
+L OtterCastAudioV2-rescue:+3.3V-S3-OLinuXino_Rev_A #PWR0105
 U 1 1 62FAA3E6
 P 11050 7850
@@
 	10450 3300 10450 3350
 $Comp
-L otter:GND #PWR0106
+L OtterCastAudioV2-rescue:GND-otter #PWR0106
 U 1 1 632DD215
 P 10450 3550
@@
 $EndComp
 $Comp
-L otter:GND #PWR0107
+L OtterCastAudioV2-rescue:GND-otter #PWR0107
 U 1 1 635CE777
 P 6800 9100
@@
 UART1_RX
 $Comp
-L S3-OLinuXino_Rev_A:+3.3V #PWR0108
+L OtterCastAudioV2-rescue:+3.3V-S3-OLinuXino_Rev_A #PWR0108
 U 1 1 63623CC5
 P 6800 9400
@@
 MIPI-PWDN
 $Comp
-L S3-OLinuXino_Rev_A:+3.3V #PWR0109
+L OtterCastAudioV2-rescue:+3.3V-S3-OLinuXino_Rev_A #PWR0109
 U 1 1 63B28C18
 P 4050 5750
@@
 NoConn ~ 6750 2300
 $Comp
-L otter:AllWinner-S3(FBGA-234) U1
+L OtterCastAudioV2-rescue:AllWinner-S3(FBGA-234)-otter U1
 U 1 1 67AEEB6A
 P 5450 2900
@@
 $EndComp
 $Comp
-L otter:AllWinner-S3(FBGA-234) U1
+L OtterCastAudioV2-rescue:AllWinner-S3(FBGA-234)-otter U1
 U 3 1 67AF4AB4
 P 5450 6400
@@
 GPIO_LED2
 $Comp
-L S3-OLinuXino_Rev_A:GND #PWR0111
+L OtterCastAudioV2-rescue:GND-S3-OLinuXino_Rev_A #PWR0111
 U 1 1 67BFC606
 P 8450 10700
@@
 MIPI-MSCK
 $Comp
-L otter:AllWinner-S3(FBGA-234) U1
+L OtterCastAudioV2-rescue:AllWinner-S3(FBGA-234)-otter U1
 U 2 1 67AFCAD8
 P 12350 4500
@@
 $EndComp
 $Comp
-L S3-OLinuXino_Rev_A:+3.3V #PWR0154
+L OtterCastAudioV2-rescue:+3.3V-S3-OLinuXino_Rev_A #PWR0154
 U 1 1 5FCE77D5
 P 7700 9250
