File: Power.sch (KiCad schematic (older format))
At the start: 80 parts, among them J3 USB, J4 OTG, Q1 DTA114YKA, SW3 RST, U1 AllWinner-S3(FBGA-234), U3 AXP209(QFN-48), U4 SY8089AAAC, U5 SY6280AAC

Commit message: Implement battery management
Very rough and needs some clenup
Parts:
- removed C15: 100n, otter:C_0402, symbol Device:C_Small
- removed R19, R20: 2.2k, otter:R_0402, symbol Device:R_Small
- added C40, C80: 10u, otter:C_0603, symbol Device:C_Small
- added L6: 2.2uH, Inductor_SMD:L_Taiyo-Yuden_MD-3030, symbol Device:L_Small
- added R5: 0R, otter:R_0805, symbol Device:R_Small
- added TP1: BAT+, TestPoint:TestPoint_THTPad_D1.5mm_Drill0.7mm, symbol Connector:TestPoint
- J3: symbol Connector:USB_C_Receptacle_USB2.0 -> OtterCastAudioV2-rescue:USB_C_Receptacle_USB2.0-Connector
- U1: symbol otter:AllWinner-S3(FBGA-234) -> OtterCastAudioV2-rescue:AllWinner-S3(FBGA-234)-otter
- U3: symbol otter:AXP209(QFN-48) -> OtterCastAudioV2-rescue:AXP209(QFN-48)-otter
- U4: symbol S3-OLinuXino_Rev_A:SY8009AAAC(SOT23-5) -> OtterCastAudioV2-rescue:SY8009AAAC(SOT23-5)-S3-OLinuXino_Rev_A
- U5: symbol otter:SY6280AAC -> OtterCastAudioV2-rescue:SY6280AAC-otter
Connections:
- net labels added: MIPI-SCK, MIPI-SDA
- net labels removed: PB6\TWI0-SCK, PB7\TWI0-SDA
- wire segments 311 -> 321
- no-connect marks 9 -> 7
