File: WifiBT.sch (KiCad schematic (older format))
At the start: 28 parts, among them U7 AP6236, X1 26Mhz TCXO

Commit message: Implement battery management
Very rough and needs some clenup
Parts:
- AE1: symbol otter:KH-5220-A56_U.FL -> OtterCastAudioV2-rescue:KH-5220-A56_U.FL-otter
- U7: symbol otter:AP6236 -> OtterCastAudioV2-rescue:AP6236-otter
Changed lines of the file:
@@
 $EndDescr
 $Comp
-L S3-OLinuXino_Rev_A:+3.3V #PWR?
+L OtterCastAudioV2-rescue:+3.3V-S3-OLinuXino_Rev_A #PWR?
 U 1 1 61C2BFBC
 P 6150 2500
@@
 $EndComp
 $Comp
-L S3-OLinuXino_Rev_A:+3.3V #PWR?
+L OtterCastAudioV2-rescue:+3.3V-S3-OLinuXino_Rev_A #PWR?
 U 1 1 67FA8CCD
 P 7750 4750
@@
 $EndComp
 $Comp
-L S3-OLinuXino_Rev_A:+3.3V #PWR?
+L OtterCastAudioV2-rescue:+3.3V-S3-OLinuXino_Rev_A #PWR?
 U 1 1 67FAEE07
 P 7750 4350
@@
 	7600 5050 7750 5050
 $Comp
-L S3-OLinuXino_Rev_A:GND #PWR?
+L OtterCastAudioV2-rescue:GND-S3-OLinuXino_Rev_A #PWR?
 U 1 1 67FBF5AE
 P 4700 3600
@@
 Connection ~ 2200 4150
 $Comp
-L S3-OLinuXino_Rev_A:GND #PWR?
+L OtterCastAudioV2-rescue:GND-S3-OLinuXino_Rev_A #PWR?
 U 1 1 67FD8D22
 P 2200 4400
@@
 $EndComp
 $Comp
-L S3-OLinuXino_Rev_A:GND #PWR?
+L OtterCastAudioV2-rescue:GND-S3-OLinuXino_Rev_A #PWR?
 U 1 1 67FDA7B2
 P 1850 4400
@@
 $EndComp
 $Comp
-L S3-OLinuXino_Rev_A:GND #PWR?
+L OtterCastAudioV2-rescue:GND-S3-OLinuXino_Rev_A #PWR?
 U 1 1 67FDC2CD
 P 1750 4000
@@
 	4100 3550 4100 3500
 $Comp
-L S3-OLinuXino_Rev_A:+3.3V #PWR?
+L OtterCastAudioV2-rescue:+3.3V-S3-OLinuXino_Rev_A #PWR?
 U 1 1 67FE9364
 P 4050 3250
@@
 Connection ~ 4100 3250
 $Comp
-L S3-OLinuXino_Rev_A:GND #PWR?
+L OtterCastAudioV2-rescue:GND-S3-OLinuXino_Rev_A #PWR?
 U 1 1 67FED111
 P 4050 3550
@@
 	2900 3400 2900 3350
 $Comp
-L S3-OLinuXino_Rev_A:+3.3V #PWR?
+L OtterCastAudioV2-rescue:+3.3V-S3-OLinuXino_Rev_A #PWR?
 U 1 1 67FF37F7
 P 2850 3100
@@
 Connection ~ 2900 3100
 $Comp
-L S3-OLinuXino_Rev_A:GND #PWR?
+L OtterCastAudioV2-rescue:GND-S3-OLinuXino_Rev_A #PWR?
 U 1 1 67FF37FF
 P 2850 3400
@@
 	6150 3950 5950 3950
 $Comp
-L otter:KH-5220-A56_U.FL AE1
+L OtterCastAudioV2-rescue:KH-5220-A56_U.FL-otter AE1
 U 1 1 60E512A9
 P 1850 3800
@@
 NoConn ~ 1950 4000
 $Comp
-L otter:AP6236 U7
+L OtterCastAudioV2-rescue:AP6236-otter U7
 U 1 1 5FD28761
 P 5350 4150
@@
 $EndComp
 $Comp
-L S3-OLinuXino_Rev_A:GND #PWR?
+L OtterCastAudioV2-rescue:GND-S3-OLinuXino_Rev_A #PWR?
 U 1 1 5FDF6E60
 P 4700 5300
@@
 Connection ~ 4350 5050
 $Comp
-L S3-OLinuXino_Rev_A:GND #PWR?
+L OtterCastAudioV2-rescue:GND-S3-OLinuXino_Rev_A #PWR?
 U 1 1 5FE117F3
 P 4350 5300
@@
 $EndComp
 $Comp
-L S3-OLinuXino_Rev_A:+3.3V #PWR?
+L OtterCastAudioV2-rescue:+3.3V-S3-OLinuXino_Rev_A #PWR?
 U 1 1 5FE304F3
 P 3250 4450
@@
 NoConn ~ 4750 4650
 $Comp
-L S3-OLinuXino_Rev_A:GND #PWR?
+L OtterCastAudioV2-rescue:GND-S3-OLinuXino_Rev_A #PWR?
 U 1 1 5FE412EC
 P 3250 5050
